Commit message: first update

File: prbt_support/urdf/simple_gripper_brackets.urdf.xacro (robot description, xacro)
@@ -71,5 +71,5 @@
             <box size="${size_x} ${size_y} ${size_z}"/>
           </geometry>
-          <material name="dark_grey">
+          <material name="dark_grey_gripper">
             <color rgba="0.8 0.8 0.8 1"/>
           </material>
